File: Lab 7.kicad_sch (KiCad schematic)
At the start: 37 parts, among them IC1 TPS2832D, Q1 CSD18534KCS, Q2 CSD18534KCS, U1 TLV2372

Commit message: stuff
Parts:
- added H1, H2, H3, H4: MountingHole, MountingHole:MountingHole_3.2mm_M3, symbol Mechanical:MountingHole
- 10VD1: renamed from 10VD; footprint (none) -> Connector_Phoenix_MSTB:PhoenixContact_MSTBA_2,5_2-G_1x02_P5.00mm_Horizontal
- 10V_T2, GND_T1, GND_T2, GND_T3, GND_T4, GND_T5, GND_T6, GND_T7, GND_T8, LOWDR_T4, LOW_Vds_T5, OPAMP_OUT_T8, PWM_T3, V_1L_T7, Vin_T1, Vout_T6: footprint (none) -> TestPoint:TestPoint_Keystone_5010-5014_Multipurpose
- C1, C2, C3, C4, C5, C6, C7: footprint (none) -> Capacitor_THT:C_Disc_D3.8mm_W2.6mm_P2.50mm
- IC1: footprint SamacSys_Parts:SOIC127P600X175-8N -> Package_SO:SO-8_3.9x4.9mm_P1.27mm
- L1: footprint SamacSys_Parts:7447231101 -> BuckParts:7447231101
- PWM1: footprint (none) -> Connector_Coaxial:BNC_Amphenol_B6252HB-NPP3G-50_Horizontal
- Q1, Q2: footprint SamacSys_Parts:TO254P470X1016X2016-3P -> Package_TO_SOT_THT:TO-220-3_Vertical
- R1, R2, R4, R5: footprint (none) -> Resistor_THT:R_Axial_DIN0207_L6.3mm_D2.5mm_P10.16mm_Horizontal
- R3: footprint (none) -> Resistor_THT:R_Axial_DIN0922_L20.0mm_D9.0mm_P30.48mm_Horizontal
- U1: footprint (none) -> Package_SO:SO-8_3.9x4.9mm_P1.27mm
- Vin1, Vout1: footprint (none) -> Connector_Phoenix_MSTB:PhoenixContact_MSTBA_2,5_2-G_1x02_P5.00mm_Horizontal
Connections:
- net Vout-: now also U1.3 (+)
